File: USBHopper.brd (EAGLE design)
At the start: 79.8 x 20.3 mm, 38 parts, among them X1 USB-1X-2S-PLUG-A-SMD

Commit message: LED Steuerung via RN4904
Parts:
- removed R2: 270, rcl:R0805
- removed TXLED: Rot, led:CHIP-LED0805
- added JRX, JTX: (no value), flo-parts:0805_CONNECT
- added R11: 270, rcl:R0805
- added TXLED2: Rot, led:CHIP-LED0805
- added U$32, U$46: (no value), flo-logic:SOT-363
- T4: device transistor:SOT23-BEC -> transistor:SOT23-EBC
- TXLED1: value Grün -> Rot
- moved R1 9.53 mm to (50.8, 17.8)
- moved T4 8.84 mm to (31.8, 6.35)
- moved JVINT 0.63 mm to (40.6, 17.8)
- renumbered RXLED to TXLED1
Connections:
- new net N$10: JTX.P$1, TXLED1.C, U$32.P$3
- new net N$11: R11.1, TXLED1.A
- new net N$12: R1.1, TXLED2.A
- new net N$9: U$32.P$1, U$32.P$5
- new net RX: U$46.P$2
- new net TX: U$32.P$2
- net +5V: now also R1.2, R11.2
- net GND: now also T4.E, U$32.P$4, U$46.P$4; no longer T4.C
- net N$5: now also U$46.P$1, U$46.P$5; no longer R1.1, TXLED1.A
- net N$6: now also JRX.P$1, TXLED2.C, U$46.P$3; no longer R2.1, TXLED.A
- net RXLED#: now also JRX.P$2; no longer TXLED1.C
- net SENSLED: now also T4.C; no longer T4.E
- net TXLED#: now also JTX.P$2; no longer TXLED.C
- net VCCIO: now also U$32.P$6, U$46.P$6; no longer R1.2, R2.2

Commit message: pnp/npn package groesser. strom schaltung gefummele.
Parts:
- removed JVINT: 0, rcl:R0805
- removed R10: 10k, rcl:R0805
- removed R6: 100k, rcl:R0805
- removed T4: (no value), transistor:SOT23-EBC
- removed TXLED2: Rot, led:CHIP-LED0805
- removed U$2: IRLML6402, IRLML6402:SOT-23
- added IC1: (no value), ic-package:DIL08
- added JINT: (no value), flo-parts:0805_CONNECT
- added RXLED: Rot, led:CHIP-LED0805
- added U$57: DMP2240UDM, flo-logic:SOT-26
- added U$64, U$72: 4k7/47k, flo-logic:SOT-457
- added U$73: (no value), flo-logic:SOT-457
- U$32, U$46: value (none) -> CON1X4; device flo-logic:SOT-363 -> flo-header:1X4PINS
- moved R5 19.0 mm to (48.3, 2.54)
- moved RS485 14.6 mm to (44.5, 10.2)
- moved U$32 12.6 mm to (48.3, 8.89), turned to 0 degrees
- moved U$46 11.3 mm to (40.6, 8.89), turned to 0 degrees
- moved HSENSE 10.8 mm to (36.8, 2.54)
- moved FTDI 8.26 mm to (56.5, 10.2)
- moved JTX 8.25 mm to (48.9, 17.8), flipped to the top
- moved HGND 6.98 mm to (24.8, 19.1)
- moved CX 6.35 mm to (37.5, 17.8)
- moved JRX 5.08 mm to (42.5, 17.8), flipped to the top
- moved R1 3.81 mm to (54.6, 17.8)
- moved R11 3.18 mm to (57.1, 17.8)
- moved R3 3.18 mm to (57.1, 2.54)
- moved SENSE 3.18 mm to (60.3, 2.54)
- moved C5 2.54 mm to (34.3, 10.2)
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- renumbered TXLED1 to TXLED
Connections:
- removed net N$23: R10.1, T4.B
- net +3V3: now also JINT.P$2; no longer JVINT.1
- net +3V3OUT: now also JINT.P$1; no longer JVINT.2
- net +5V: now also U$32.P$1, U$57.P$6; no longer U$2.3, U$20.P1, U$20.P3, U$49.P$2
- net DI: now also U$46.P$4
- net GND: now also U$64.P$6, U$72.P$6, U$73.P$6; no longer R6.2, T4.E, U$46.P$4
- net N$10: now also U$64.P$1; no longer U$32.P$3
- net N$12: now also RXLED.A; no longer TXLED2.A
- net N$5: now also U$72.P$2, U$72.P$3; no longer U$46.P$1, U$46.P$5
- net N$6: now also RXLED.C, U$72.P$1; no longer TXLED2.C, U$46.P$3
- net N$9: now also U$64.P$2, U$64.P$3; no longer U$32.P$1, U$32.P$5
- net PWREN: now also U$57.P$1; no longer U$2.1
- net PWREN#: now also U$46.P$2
- net RO: now also U$46.P$1
- net RS485A: now also U$32.P$2
- net RS485B: now also U$32.P$3
- net RX: now also U$72.P$5; no longer U$46.P$2
- net SENSE: now also U$73.P$2; no longer R10.2, R6.1
- net SENSLED: now also U$73.P$1; no longer T4.C
- net TX: now also U$64.P$5; no longer U$32.P$2
- net TXDEN: now also U$46.P$3
- net USB+5V: now also U$20.P1, U$20.P3, U$49.P$2, U$57.P$5; no longer U$2.2
- net VCCIO: now also U$64.P$4, U$72.P$4; no longer U$32.P$6, U$46.P$6
Routing:
- net USB+5V: track 27.3 -> 37.7 mm, vias 2 -> 4
- net +5V: track 13.8 -> 9.05 mm, vias 4 -> 2
- net N$1: track 2.55 -> 5.72 mm
Other:
- board text removed: "T"

Commit message: weiter pwren, leds...
Parts:
- removed IC1: (no value), ic-package:DIL08
- removed JINT: (no value), flo-parts:0805_CONNECT
- removed R5: 0, rcl:R0805
- removed U$64: 4k7/47k, flo-logic:SOT-457
- added JP1, JP2: (no value), pinhead:1X01
- added UTX: 4k7/47k, flo-logic:SOT-457
- C5: device rcl:PANASONIC_B -> rcl:153CLV-0405
- PWRLED: value Orange -> Blue
- RXLED: value Rot -> Red
- TXLED: value Rot -> Green
- moved C4 21.7 mm to (52.1, 12.7)
- moved JRX 18.8 mm to (59.7, 10.2), flipped to the bottom
- moved JTX 14.8 mm to (61.6, 10.2), flipped to the bottom
- moved CX 12.8 mm to (24.8, 15.9), turned to 180 degrees
- moved C5 2.54 mm to (31.8, 10.2)
- moved FTDI 2.54 mm to (59.1, 10.2)
- moved U$57 2.54 mm to (14.0, 12.7)
- moved RS485 1.27 mm to (43.2, 10.2)
- moved U$46 1.27 mm to (39.4, 8.89)
- moved U$32 1.27 mm to (47.0, 8.89)
- renumbered R1 to RRX, R11 to RTX, U$72 to URX
Connections:
- new net N$13: R3.2, U$73.P$3
- new net N$14: JP1.1, U$73.P$5
- net +3V3: no longer JINT.P$2
- net +3V3OUT: now also JPWRSEL.1; no longer JINT.P$1
- net +5V: now also U$20.P1, U$20.P3, U$49.P$2
- net DCD#: no longer R5.2
- net GND: now also UTX.P$6; no longer U$64.P$6
- net N$10: now also UTX.P$1; no longer U$64.P$1
- net N$9: now also UTX.P$2, UTX.P$3; no longer U$64.P$2, U$64.P$3
- net PWREN#: now also JP2.1
- net SENSLED: no longer R5.1
- net TX: now also UTX.P$5; no longer U$64.P$5
- net USB+5V: now also U$73.P$4; no longer U$20.P1, U$20.P3, U$49.P$2
- net VCCIO: now also UTX.P$4; no longer R3.2, U$64.P$4
Routing:
- net USB+5V: track 37.7 -> 28.4 mm, vias 4 -> 2
- net +5V: track 9.05 -> 13.8 mm, vias 2 -> 4
- net PWREN: track 5.70 -> 2.54 mm
Other:
- board text added: "+1v8"
- board text added: "+3v3"
- board text added: "+5v"
- board text added: "usb+5v"
- board text added: "vccio"

Commit message: +5V->USB+5V bei sense
Connections:
- net +5V: no longer R4.2
- net USB+5V: now also R4.2
Changed lines of the file:
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@@
 <wire x1="10.16" y1="13.8" x2="8.255" y2="15.705" width="0.508" layer="1"/>
 <contactref element="U$73" pad="P$4"/>
+<contactref element="R4" pad="2"/>
 <wire x1="52.07" y1="11.85" x2="60.03" y2="13.785" width="0" layer="19" extent="1-1"/>
 <wire x1="13.97" y1="10.16" x2="13.97" y2="8.001" width="0" layer="19" extent="1-1"/>
 <wire x1="12.57" y1="12.7" x2="11.43" y2="13.716" width="0" layer="19" extent="1-1"/>
-<wire x1="45.985" y1="3.74" x2="52.07" y2="11.85" width="0" layer="19" extent="1-1"/>
+<wire x1="54.61" y1="3.39" x2="52.07" y2="11.85" width="0" layer="19" extent="1-1"/>
+<wire x1="45.985" y1="3.74" x2="54.61" y2="3.39" width="0" layer="19" extent="1-1"/>
 </signal>
 <signal name="+3V3OUT">
@@
 </signal>
 <signal name="+5V">
-<contactref element="R4" pad="2"/>
 <contactref element="RS485" pad="8"/>
 <contactref element="JPWRSEL" pad="5"/>
@@
 <via x="12.954" y="14.859" extent="1-16" drill="0.5"/>
 <wire x1="12.954" y1="18.796" x2="12.954" y2="14.859" width="0.508" layer="16"/>
-<wire x1="45.085" y1="7.56" x2="54.61" y2="3.39" width="0" layer="19" extent="1-1"/>
 <wire x1="46.99" y1="13.97" x2="45.085" y2="7.56" width="0" layer="19" extent="1-1"/>
 <wire x1="23.495" y1="7.62" x2="45.085" y2="7.56" width="0" layer="19" extent="1-1"/>

Commit message: Viel Layout
Parts:
- removed C1: 10nF, rcl:C0805
- removed C3: 100nF, rcl:C0805
- removed HSENSE, JP1, JP2: (no value), pinhead:1X01
- removed U$46: CON1X4, flo-header:1X4PINS
- added C2: 10nF, flo-parts:0805
- added Q1: 2.5A/30V, SparkFun-DiscreteSemi:SOT23-3
- added U$21: CON1X1PIN_XL, flo-header:1X1PINS
- added U$27: CON1X2PIN_BRIDGE, flo-header:1X2PINS_BRIDGE
- added U$64: CON1X8PIN_L, flo-header:1X8PINS_L
- added U$66: PAD2X8PADS, flo-header:2X8PADS
- C4, CX: device rcl:C0805 -> flo-parts:0805
- R3, R4, R7, REN, RRX, RTX: device rcl:R0805 -> flo-parts:0805
- U$19: value PAD2X8 -> CON2X2PIN_L; device flo-header:2X8PADS -> flo-header:2X2PINS_L
- U$32: value CON1X4 -> 100nF; device flo-header:1X4PINS -> flo-parts:0805
- U$57: value DMP2240UDM -> IC8DIL; device flo-logic:SOT-26 -> flo-gen-ic:DIL8
- U$65: value CON4X8 -> PAD2X8PIN_L; device flo-header:4X8PINS -> flo-header:2X8PINS_L
- moved U$19 46.3 mm to (34.3, 3.17), turned to 90 degrees
- moved U$57 29.3 mm to (43.2, 10.2), turned to 0 degrees
- moved U$32 28.6 mm to (18.4, 10.2)
- moved JRX 12.7 mm to (49.5, 17.8)
- moved U$73 11.4 mm to (56.5, 2.54)
- moved RXLED 9.53 mm to (50.8, 17.8)
- moved SENSE 9.53 mm to (50.8, 2.54)
- moved CX 8.13 mm to (29.8, 9.53), turned to 90 degrees
- moved JTX 7.62 mm to (61.6, 17.8), turned to 270 degrees
- moved R4 6.35 mm to (48.3, 2.54)
- moved RRX 6.35 mm to (48.3, 17.8)
- moved UTX 5.72 mm to (56.5, 17.8)
- moved R3 3.18 mm to (60.3, 2.54), turned to 270 degrees
- moved RTX 3.18 mm to (60.3, 17.8)
- moved C4 2.54 mm to (52.6, 10.2)
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Connections:
- removed net FB: U$11.P4, U$51.P$1
- removed net SW: L3.P$2, U$11.P5
- net +1V8: now also U$11.P5, U$64.P$4, U$66.P$7; no longer U$19.P$8, U$65.P$16
- net +3V3: now also U$10.P$1, U$20.P5, U$64.P$3, U$66.P$5; no longer U$10.P$2, U$19.P$6, U$65.P$12
- net +3V3OUT: now also CX.P$2; no longer CX.2
- net +5V: now also Q1.3, RRX.P$2, RTX.P$2, U$32.P$2, U$57.P$8, U$64.P$2, U$66.P$3; no longer C3.1, RRX.2, RTX.2, U$19.P$4, U$32.P$1, U$57.P$6, U$65.P$8
- net CBUS4: now also U$65.P$13; no longer U$65.P$17
- net CTS#: now also U$65.P$4, U$66.P$4; no longer U$19.P$3, U$65.P$14, U$65.P$7
- net DCD#: now also U$65.P$7; no longer U$65.P$26
- net DI: now also U$19.P$4, U$57.P$4; no longer U$19.P$9, U$46.P$4, U$65.P$19
- net DSR#: now also U$65.P$6; no longer U$65.P$22
- net DTR#: now also U$65.P$5; no longer U$65.P$18
- net GND: now also C2.P$2, C4.P$1, CX.P$1, U$10.P$2, U$51.P$1, U$57.P$5, U$64.P$1, U$64.P$8, U$65.P$14, U$66.P$1, U$66.P$15; no longer C1.2, C4.2, CX.1, U$19.P$16, U$19.P$2, U$32.P$4, U$65.P$32, U$65.P$4
- net N$1: now also R3.P$1; no longer R3.1
- net N$11: now also RTX.P$1; no longer RTX.1
- net N$12: now also RRX.P$1; no longer RRX.1
- net N$13: now also R3.P$2; no longer R3.2
- net N$14: now also U$27.P$1; no longer JP1.1
- net N$2: now also R4.P$1; no longer R4.1
- net N$4: now also C2.P$1; no longer C1.1
- net N$7: now also L3.P$2, U$11.P4; no longer L2.P$2, U$20.P5
- net N$8: now also L2.P$2; no longer U$10.P$1
- net PWREN: now also Q1.1, REN.P$2, U$32.P$1; no longer C3.2, REN.1, U$57.P$1
- net PWREN#: now also R7.P$1, REN.P$1, U$27.P$2, U$57.P$2, U$65.P$12, U$66.P$6; no longer JP2.1, R7.2, REN.2, U$19.P$5, U$46.P$2, U$65.P$11, U$65.P$13
- net RI#: now also U$65.P$8; no longer U$65.P$30
- net RO: now also U$19.P$2, U$57.P$1; no longer U$19.P$11, U$46.P$1, U$65.P$23
- net RS485A: now also U$57.P$6, U$65.P$15, U$66.P$16; no longer U$19.P$15, U$32.P$2, U$65.P$31
- net RS485B: now also U$57.P$7, U$65.P$16, U$66.P$14; no longer U$19.P$13, U$32.P$3, U$65.P$27
- net RTS#: now also U$66.P$2; no longer U$19.P$1, U$65.P$10
- net RXD: now also U$19.P$1, U$64.P$6, U$65.P$2, U$66.P$11; no longer U$19.P$12, U$65.P$24, U$65.P$6
- net RXLED#: now also U$65.P$10; no longer U$65.P$5
- net SENSE: now also U$21.P$1; no longer HSENSE.1
- net TXD: now also U$19.P$3, U$64.P$5, U$65.P$1, U$66.P$9; no longer U$19.P$10, U$65.P$2, U$65.P$20
- net TXDEN: now also U$57.P$3, U$65.P$11, U$66.P$8; no longer U$19.P$7, U$46.P$3, U$65.P$15, U$65.P$9
- net TXLED#: now also U$65.P$9; no longer U$65.P$1
- net USB+5V: now also C4.P$2, Q1.2, R4.P$2, R7.P$2; no longer C4.1, R4.2, R7.1, U$57.P$5
- net VCCIO: now also U$64.P$7, U$66.P$13; no longer U$19.P$14, U$65.P$28
Routing:
- net RXD: track 3.17 -> 76.9 mm, vias 0 -> 2
- net TXD: track 3.17 -> 75.0 mm, vias 0 -> 4
- net PWREN#: track 42.9 -> 96.4 mm, vias 1 -> 7
- net TXDEN: track 8.94 -> 58.7 mm, vias 0 -> 4
- net +3V3OUT: track 0.00 -> 46.9 mm, vias 0 -> 2
- net GND: track 8.14 -> 51.7 mm, vias 51 -> 61
- net RS485B: track 9.12 -> 52.3 mm, vias 0 -> 1
- net VCCIO: track 8.41 -> 49.6 mm, vias 0 -> 8
- net USB+5V: track 28.4 -> 66.1 mm, vias 2 -> 8
- net RS485A: track 9.10 -> 45.4 mm, vias 0 -> 3
- net RXLED#: track 0.00 -> 36.3 mm, vias 0 -> 3
- net N$14: track 0.00 -> 31.4 mm, vias 0 -> 1
- net TXLED#: track 0.00 -> 27.9 mm, vias 0 -> 4
- net RTS#: track 9.05 -> 35.7 mm, vias 0 -> 1
- net +5V: track 13.8 -> 39.9 mm
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Other:
- board size 79.8 x 20.3 mm -> 85 x 20.3 mm

Commit message: Layout fertig. Logo!
Parts:
- removed CX, U$32: 100nF, flo-parts:0805
- removed RRX, RTX: 270, flo-parts:0805
- removed U$73: (no value), flo-logic:SOT-457
- removed URX, UTX: 4k7/47k, flo-logic:SOT-457
- added C1: 10nF, flo-parts:0805
- added C3: 100nF, flo-parts:0805
- added R5, R6: 270, flo-parts:0805
- added U1: (no value), flo-logic:SOT-457
- added U2, U3: 4k7/47k, flo-logic:SOT-457
- C2: value 10nF -> 100nF
- FTDI: device ftdichip:SSOP28 -> ftdichip:SSOP28_FLO
- L1: device wuerth-elektronik:0805 -> wuerth_elektronik:0805
- PWRLED, RXLED, SENSE, TXLED: device led:CHIP-LED0805 -> flo-led:KPT-2012
- U$27: value CON1X2PIN_BRIDGE -> CON1X2PIN_XL; device flo-header:1X2PINS_BRIDGE -> flo-header:1X2PINS
- moved C4 22.7 mm to (29.8, 9.53)
- moved R3 14.0 mm to (46.4, 2.54), turned to 90 degrees
- moved R4 10.2 mm to (58.4, 2.54), turned to 270 degrees
- moved C2 8.64 mm to (18.4, 10.2), turned to 0 degrees
- moved U$64 3.81 mm to (74.3, 10.2)
- moved U$65 3.81 mm to (69.8, 10.2)
- moved U$66 3.81 mm to (80.8, 10.2)
- moved FTDI 1.91 mm to (57.1, 10.2)
- moved PWRLED 1.91 mm to (61.0, 2.54)
- moved TXLED 1.91 mm to (61.0, 17.8)
- moved RXLED 1.90 mm to (48.9, 17.8)
- moved SENSE 1.90 mm to (48.9, 2.54), turned to 180 degrees
- moved C5 0.63 mm to (33.7, 10.2)
- moved RS485 0.63 mm to (42.5, 10.2)
- moved U$19 0.63 mm to (33.7, 3.17)
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- renumbered R7 to R1, REN to R2, U$10 to C8, U$11 to U5, U$20 to U4, U$35 to C7, U$49 to C6, U$51 to C9
Connections:
- removed net N$5: URX.P$2, URX.P$3
- new net U3: U3.P$2, U3.P$3
- net +3V3OUT: now also C4.P$2; no longer CX.P$2
- net +5V: now also C2.P$2, R5.P$2, R6.P$2; no longer RRX.P$2, RTX.P$2, U$32.P$2
- net GND: now also C1.P$2, C3.P$1, PWRLED.2, U1.P$6, U2.P$6, U3.P$6; no longer C2.P$2, CX.P$1, PWRLED.C, U$73.P$6, URX.P$6, UTX.P$6
- net N$1: now also PWRLED.1, R4.P$1; no longer PWRLED.A, R3.P$1
- net N$10: now also TXLED.2, U2.P$1; no longer TXLED.C, UTX.P$1
- net N$11: now also R5.P$1, TXLED.1; no longer RTX.P$1, TXLED.A
- net N$12: now also R6.P$1, RXLED.1; no longer RRX.P$1, RXLED.A
- net N$13: now also R4.P$2, U1.P$3; no longer R3.P$2, U$73.P$3
- net N$14: now also U1.P$5; no longer U$73.P$5
- net N$2: now also R3.P$1, SENSE.1; no longer R4.P$1, SENSE.A
- net N$4: now also C1.P$1; no longer C2.P$1
- net N$6: now also RXLED.2, U3.P$1; no longer RXLED.C, URX.P$1
- net N$9: now also U2.P$2, U2.P$3; no longer UTX.P$2, UTX.P$3
- net PWREN: now also C2.P$1; no longer U$32.P$1
- net RX: now also U3.P$5; no longer URX.P$5
- net SENSE: now also U1.P$2; no longer U$73.P$2
- net SENSLED: now also SENSE.2, U1.P$1; no longer SENSE.C, U$73.P$1
- net TX: now also U2.P$5; no longer UTX.P$5
- net USB+5V: now also C3.P$2, R3.P$2, U1.P$4; no longer C4.P$2, R4.P$2, U$73.P$4
- net VCCIO: now also U2.P$4, U3.P$4; no longer URX.P$4, UTX.P$4
Routing:
- net VCCIO: track 49.6 -> 62.4 mm, vias 8 -> 11
- net PWREN#: track 96.4 -> 92.6 mm
- net RXLED#: track 36.3 -> 32.5 mm
- net RXD: track 76.9 -> 73.5 mm
- net TXDEN: track 58.7 -> 55.4 mm
- net TXD: track 75.0 -> 71.8 mm
- net RS485B: track 52.3 -> 54.7 mm, vias 1 -> 2
- net CTS#: track 32.2 -> 30.3 mm
- net RI#: track 19.3 -> 17.4 mm
- net DTR#: track 21.1 -> 19.2 mm
- net DCD#: track 15.2 -> 13.3 mm
- net CBUS4: track 12.6 -> 10.7 mm
- net USBDP: track 61.3 -> 59.4 mm
- net RTS#: track 35.7 -> 33.8 mm
- net N$14: track 31.4 -> 29.5 mm
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Other:
- board size 85 x 20.3 mm -> 81.2 x 20.3 mm
- board text added: "+ B A -"
- board text added: "1"
- board text added: "14"
- board text added: "15"
- board text added: "1v8"
- board text added: "2"
- board text added: "28"
- board text added: "3"
- board text added: "3v3"
- board text added: "4"
- board text added: "42"
- board text added: "485"
- board text added: "5"
- board text added: "8"
- board text added: "=HOT="
- board text added: "?"
- board text added: "All Rights Reversed"
- board text added: "BETA"
- board text added: "C1"
- board text added: "C2"
- board text added: "C3"
- board text added: "C4"
- board text added: "C5"
- board text added: "C6"
- board text added: "C7"
- board text added: "C8"
- board text added: "C9"
- board text added: "DI"
- board text added: "DM"
- board text added: "DP"
- board text added: "ENTER YOUR NAME HERE"
- board text added: "GND"
- board text added: "HOT END"
- board text added: "L1"
- board text added: "L2"
- board text added: "L3"
- board text added: "MOTHER BOARD"
- board text added: "NOW YOU SEE ME"
- board text added: "PUNK"
- board text added: "R1"
- board text added: "R2"
- board text added: "R3"
- board text added: "R4"
- board text added: "R5"
- board text added: "R6"
- board text added: "RO"
- board text added: "RO RE DE DI"
- board text added: "RXD CTS DSR RI CB1 CB3 GND B"
- board text added: "S"
- board text added: "TXD RTS DTR DCD CB0 CB2 CB4 A"
- board text added: "U1"
- board text added: "U2"
- board text added: "U3"
- board text added: "U4"
- board text added: "U5"
- board text added: "VCC"
- board text added: "binary"
- board text added: "is not"
- board text added: "kitchen"
- board text added: "www.binary-kitchen.de"
- board text removed: "+1v8"
- board text removed: "+3v3"
- board text removed: "+5v"
- board text removed: "- +"
- board text removed: "INT"
- board text removed: "usb+5v"
- board text removed: "vccio"
