File: USBHopper.sch (EAGLE design)
At the start: 42 parts, among them Q1 2.5A/30V, U2 4k7/47k, U3 4k7/47k, U4 DCDC, U5 DCDC, X1 USB-1X-2S-PLUG-A-SMD

Commit message: The downside is the upside.
Parts:
- added R10, R11, R12, R9: 0, flo-parts:RESISTORCONNECT
- added R7: 60, flo-parts:RESISTORWIDE
- added R8: 60, flo-parts:RESISTORCONNECT
- added U$10, U$11, U$4, U$5: CON1X1PIN_XL, flo-header:CON1X1PIN_XL
- added U$20: TANTAL1206, flo-parts:TANTAL1206
- C5: value 4.7µF -> 220pF; device rcl:CPOL-EU153CLV-0405 -> flo-parts:CAPACITOR
- C6: value 4.4µF -> 4.7µF
- C7: value 4.4µF <- check -> 4.7µF
- C9: value 10µF <- check -> 10µF
- JRX, JTX: value (none) -> 0
- L2: value 2.2µH -> 1.0µH
- L3: value 2.2µH <- check -> 1.0µH
- R4: value 270 -> 330
- U1: value (none) -> 4k7/47k
- U4: value DCDC -> ADP2108AUJZ-3.3-R7
- U5: value DCDC -> ADP2108AUJZ-1.8-R7
Connections:
- removed net RX: U3PNP.B
- removed net TX: U2PNP.B
- removed net U3: U3NPN.B, U3PNP.C
- new net DE: R10.P$2, RS485.DE, U$57.P$3
- new net N$5: L2.P$2, U4.SW
- new net RE#: R9.P$2, RS485.!RE, U$57.P$2
- new net SEN3: U$10.P$1, U2NPN.B, U2PNP.C
- new net SEN4: U$11.P$1, U3NPN.B, U3PNP.C
- net +1V8: now also U5.FB; no longer U5.SW
- net +3V3: now also R11.P$2, U4.FB; no longer U4.SW
- net +5V: now also R12.P$2, U$4.P$1; no longer RS485.VCC, U$57.P$8
- net GND: now also C5.P$2, LED2.C$1, U$20.P$2, U$5.P$1; no longer C5.-, LED2.C
- net N$1: now also LED2.A$1; no longer LED2.A
- net N$10: now also LED4.C$1; no longer LED4.C
- net N$11: now also LED4.A$1; no longer LED4.A
- net N$12: now also LED3.A$1; no longer LED3.A
- net N$2: now also LED1.A$1; no longer LED1.A
- net N$6: now also LED3.C$1; no longer LED3.C
- net N$7: now also U5.SW; no longer U5.FB
- net N$8: now also C5.P$1, R7.P$1, R8.P$1; no longer L2.P$2, U4.FB
- net N$9: now also R11.P$1, R12.P$1, RS485.VCC, U$57.P$8; no longer U2NPN.B, U2PNP.C
- net PWREN#: now also R9.P$1; no longer RS485.!RE, U$57.P$2
- net RS485A: now also R7.P$2
- net RS485B: now also R8.P$2
- net RXD: now also U3PNP.B
- net SENSLED: now also LED1.C$1; no longer LED1.C
- net TXD: now also U2PNP.B
- net TXDEN: now also R10.P$1; no longer RS485.DE, U$57.P$3
- net USB+5V: now also U$20.P$1; no longer C5.+
Other:
- note added: "485EN"
- note added: "485PWR"
- note added: "FT232R"
- note added: "IO Leds + S3/4"
- note added: "POWER + decouple"
- note added: "PWR LED + S2"
- note added: "PWR Sel"
- note added: "RS485"
- note added: "S1"
- note added: "chip"
- note added: "io"
- note added: "term"
- moved on the sheet: C1, C2, C3, C4, C6, C7, C8, C9, FTDI, HGND, JRX, JTX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
