File: USBHopper.sch (EAGLE design)
At the start: 53 parts, among them Q1 2.5A/30V, U1 4k7/47k, U2 4k7/47k, U3 4k7/47k, U4 ADP2108AUJZ-3.3-R7, U5 ADP2108AUJZ-1.8-R7, X1 USB-1X-2S-PLUG-A-SMD

Commit message: Bugfixes. Pad auf GND.
Connections:
- removed net SENSLED: LED1.C$1, U1NPN.E
- new net N$15: LED1.C$1, U1NPN.C
- net GND: now also U1NPN.E, U2NPN.E, U3NPN.E; no longer U1NPN.C, U2NPN.C, U3NPN.C
- net N$10: now also U2NPN.C; no longer U2NPN.E
- net N$6: now also U3NPN.C; no longer U3NPN.E
Changed lines of the file:
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@@
 <grid distance="0.1" unitdist="inch" unit="inch" style="lines" multiple="1" display="no" altdistance="0.01" altunitdist="inch" altunit="inch"/>
 <layers>
-<layer number="1" name="Top" color="4" fill="1" visible="yes" active="no"/>
-<layer number="16" name="Bottom" color="1" fill="1" visible="yes" active="no"/>
-<layer number="17" name="Pads" color="3" fill="1" visible="yes" active="no"/>
-<layer number="18" name="Vias" color="2" fill="1" visible="yes" active="no"/>
-<layer number="19" name="Unrouted" color="6" fill="1" visible="yes" active="no"/>
-<layer number="20" name="Dimension" color="15" fill="1" visible="yes" active="no"/>
-<layer number="21" name="tPlace" color="7" fill="1" visible="yes" active="no"/>
-<layer number="22" name="bPlace" color="7" fill="1" visible="yes" active="no"/>
-<layer number="23" name="tOrigins" color="15" fill="1" visible="yes" active="no"/>
-<layer number="24" name="bOrigins" color="15" fill="1" visible="yes" active="no"/>
-<layer number="25" name="tNames" color="7" fill="1" visible="yes" active="no"/>
-<layer number="26" name="bNames" color="7" fill="1" visible="yes" active="no"/>
-<layer number="27" name="tValues" color="7" fill="1" visible="yes" active="no"/>
-<layer number="28" name="bValues" color="7" fill="1" visible="yes" active="no"/>
+<layer number="1" name="Top" color="4" fill="1" visible="no" active="no"/>
+<layer number="16" name="Bottom" color="1" fill="1" visible="no" active="no"/>
+<layer number="17" name="Pads" color="3" fill="1" visible="no" active="no"/>
+<layer number="18" name="Vias" color="2" fill="1" visible="no" active="no"/>
+<layer number="19" name="Unrouted" color="6" fill="1" visible="no" active="no"/>
+<layer number="20" name="Dimension" color="15" fill="1" visible="no" active="no"/>
+<layer number="21" name="tPlace" color="7" fill="1" visible="no" active="no"/>
+<layer number="22" name="bPlace" color="7" fill="1" visible="no" active="no"/>
+<layer number="23" name="tOrigins" color="15" fill="1" visible="no" active="no"/>
+<layer number="24" name="bOrigins" color="15" fill="1" visible="no" active="no"/>
+<layer number="25" name="tNames" color="7" fill="1" visible="no" active="no"/>
+<layer number="26" name="bNames" color="7" fill="1" visible="no" active="no"/>
+<layer number="27" name="tValues" color="7" fill="1" visible="no" active="no"/>
+<layer number="28" name="bValues" color="7" fill="1" visible="no" active="no"/>
 <layer number="29" name="tStop" color="7" fill="3" visible="no" active="no"/>
 <layer number="30" name="bStop" color="7" fill="6" visible="no" active="no"/>
@@
 <layer number="35" name="tGlue" color="7" fill="4" visible="no" active="no"/>
 <layer number="36" name="bGlue" color="7" fill="5" visible="no" active="no"/>
-<layer number="37" name="tTest" color="7" fill="1" visible="yes" active="no"/>
-<layer number="38" name="bTest" color="7" fill="1" visible="yes" active="no"/>
+<layer number="37" name="tTest" color="7" fill="1" visible="no" active="no"/>
+<layer number="38" name="bTest" color="7" fill="1" visible="no" active="no"/>
 <layer number="39" name="tKeepout" color="4" fill="11" visible="no" active="no"/>
 <layer number="40" name="bKeepout" color="1" fill="11" visible="no" active="no"/>
@@
 <layer number="44" name="Drills" color="7" fill="1" visible="no" active="no"/>
 <layer number="45" name="Holes" color="7" fill="1" visible="no" active="no"/>
-<layer number="46" name="Milling" color="3" fill="1" visible="yes" active="no"/>
-<layer number="47" name="Measures" color="7" fill="1" visible="yes" active="no"/>
-<layer number="48" name="Document" color="7" fill="1" visible="yes" active="no"/>
-<layer number="49" name="Reference" color="7" fill="1" visible="yes" active="no"/>
-<layer number="50" name="dxf" color="7" fill="1" visible="yes" active="no"/>
-<layer number="51" name="tDocu" color="14" fill="1" visible="yes" active="no"/>
-<layer number="52" name="bDocu" color="7" fill="1" visible="yes" active="no"/>
-<layer number="53" name="tGND_GNDA" color="7" fill="9" visible="yes" active="no"/>
-<layer number="54" name="bGND_GNDA" color="1" fill="9" visible="yes" active="no"/>
-<layer number="56" name="wert" color="7" fill="1" visible="yes" active="no"/>
-<layer number="57" name="tCAD" color="7" fill="1" visible="yes" active="no"/>
+<layer number="46" name="Milling" color="3" fill="1" visible="no" active="no"/>
+<layer number="47" name="Measures" color="7" fill="1" visible="no" active="no"/>
+<layer number="48" name="Document" color="7" fill="1" visible="no" active="no"/>
+<layer number="49" name="Reference" color="7" fill="1" visible="no" active="no"/>
+<layer number="50" name="dxf" color="7" fill="1" visible="no" active="no"/>
+<layer number="51" name="tDocu" color="14" fill="1" visible="no" active="no"/>
+<layer number="52" name="bDocu" color="7" fill="1" visible="no" active="no"/>
+<layer number="53" name="tGND_GNDA" color="7" fill="9" visible="no" active="no"/>
+<layer number="54" name="bGND_GNDA" color="1" fill="9" visible="no" active="no"/>
+<layer number="56" name="wert" color="7" fill="1" visible="no" active="no"/>
+<layer number="57" name="tCAD" color="7" fill="1" visible="no" active="no"/>
 <layer number="90" name="Modules" color="5" fill="1" visible="yes" active="yes"/>
 <layer number="91" name="Nets" color="2" fill="1" visible="yes" active="yes"/>
@@
 <segment>
 <pinref part="U$55" gate="G$1" pin="GND"/>
-<wire x1="-53.34" y1="-58.42" x2="-53.34" y2="-66.04" width="0.1524" layer="91"/>
 <wire x1="-53.34" y1="-66.04" x2="-66.04" y2="-66.04" width="0.1524" layer="91"/>
-<pinref part="U1" gate="NPN" pin="C"/>
+<pinref part="U1" gate="NPN" pin="E"/>
+<wire x1="-53.34" y1="-66.04" x2="-53.34" y2="-58.42" width="0.1524" layer="91"/>
 </segment>
 <segment>
@@
 </segment>
 <segment>
-<wire x1="66.04" y1="-66.04" x2="66.04" y2="-63.5" width="0.1524" layer="91"/>
 <pinref part="U$60" gate="G$1" pin="GND"/>
+<wire x1="106.68" y1="-66.04" x2="66.04" y2="-66.04" width="0.1524" layer="91"/>
+<pinref part="U3" gate="NPN" pin="E"/>
 <wire x1="66.04" y1="-66.04" x2="33.02" y2="-66.04" width="0.1524" layer="91"/>
 <wire x1="106.68" y1="-66.04" x2="106.68" y2="-63.5" width="0.1524" layer="91"/>
-<wire x1="106.68" y1="-66.04" x2="66.04" y2="-66.04" width="0.1524" layer="91"/>
+<pinref part="U2" gate="NPN" pin="E"/>
+<wire x1="66.04" y1="-63.5" x2="66.04" y2="-66.04" width="0.1524" layer="91"/>
 <junction x="66.04" y="-66.04"/>
-<pinref part="U2" gate="NPN" pin="C"/>
-<pinref part="U3" gate="NPN" pin="C"/>
 </segment>
 <segment>
@@
 </segment>
 </net>
-<net name="SENSLED" class="0">
-<segment>
-<wire x1="-53.34" y1="-43.18" x2="-53.34" y2="-45.72" width="0.1524" layer="91"/>
-<pinref part="LED1" gate="G$1" pin="C$1"/>
-<pinref part="U1" gate="NPN" pin="E"/>
-</segment>
-</net>
 <net name="DSR#" class="0">
 <segment>
@@
 <segment>
 <pinref part="LED4" gate="G$1" pin="C$1"/>
-<wire x1="66.04" y1="-50.8" x2="66.04" y2="-48.26" width="0.1524" layer="91"/>
 <pinref part="JTX" gate="R$1" pin="P$1"/>
 <wire x1="66.04" y1="-48.26" x2="66.04" y2="-45.72" width="0.1524" layer="91"/>
 <wire x1="66.04" y1="-48.26" x2="71.12" y2="-48.26" width="0.1524" layer="91"/>
 <wire x1="71.12" y1="-48.26" x2="71.12" y2="-73.66" width="0.1524" layer="91"/>
+<pinref part="U2" gate="NPN" pin="C"/>
+<wire x1="66.04" y1="-48.26" x2="66.04" y2="-50.8" width="0.1524" layer="91"/>
 <junction x="66.04" y="-48.26"/>
-<pinref part="U2" gate="NPN" pin="E"/>
 </segment>
 </net>
@@
 <segment>
 <pinref part="LED3" gate="G$1" pin="C$1"/>
-<wire x1="106.68" y1="-50.8" x2="106.68" y2="-48.26" width="0.1524" layer="91"/>
 <pinref part="JRX" gate="R$1" pin="P$1"/>
 <wire x1="106.68" y1="-48.26" x2="106.68" y2="-45.72" width="0.1524" layer="91"/>
 <wire x1="106.68" y1="-48.26" x2="111.76" y2="-48.26" width="0.1524" layer="91"/>
 <wire x1="111.76" y1="-48.26" x2="111.76" y2="-73.66" width="0.1524" layer="91"/>
+<pinref part="U3" gate="NPN" pin="C"/>
+<wire x1="106.68" y1="-48.26" x2="106.68" y2="-50.8" width="0.1524" layer="91"/>
 <junction x="106.68" y="-48.26"/>
-<pinref part="U3" gate="NPN" pin="E"/>
 </segment>
 </net>
@@
 </segment>
 </net>
+<net name="N$15" class="0">
+<segment>
+<pinref part="LED1" gate="G$1" pin="C$1"/>
+<pinref part="U1" gate="NPN" pin="C"/>
+<wire x1="-53.34" y1="-43.18" x2="-53.34" y2="-45.72" width="0.1524" layer="91"/>
+</segment>
+</net>

Commit message: V1.0
Parts:
- LED1, LED2, LED3, LED4: device flo-led:LEDKPT-2012 -> flo-led:LEDKPT-2012-E
- renumbered U$10 to S4, U$11 to S3, U$21 to S1, U$27 to S2
Changed lines of the file:
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@@
 <layer number="50" name="dxf" color="7" fill="1" visible="no" active="no"/>
 <layer number="51" name="tDocu" color="14" fill="1" visible="no" active="no"/>
-<layer number="52" name="bDocu" color="7" fill="1" visible="no" active="no"/>
+<layer number="52" name="bDocu" color="6" fill="1" visible="no" active="no"/>
 <layer number="53" name="tGND_GNDA" color="7" fill="9" visible="no" active="no"/>
 <layer number="54" name="bGND_GNDA" color="1" fill="9" visible="no" active="no"/>
@@
 <part name="U$24" library="supply3" deviceset="GND" device=""/>
 <part name="U$50" library="supply3" deviceset="+5V" device=""/>
-<part name="LED2" library="flo-led" deviceset="LED" device="KPT-2012" value="Blue"/>
+<part name="LED2" library="flo-led" deviceset="LED" device="KPT-2012-E" value="Blue"/>
 <part name="U$52" library="supply3" deviceset="GND" device=""/>
 <part name="HGND" library="pinhead" deviceset="PINHD-1X2" device=""/>
@@
 <part name="U$56" library="supply3" deviceset="GND" device=""/>
 <part name="U$58" library="supply3" deviceset="GND" device=""/>
-<part name="LED1" library="flo-led" deviceset="LED" device="KPT-2012" value="Orange"/>
+<part name="LED1" library="flo-led" deviceset="LED" device="KPT-2012-E" value="Orange"/>
 <part name="U4" library="flo-parts" deviceset="DCDC" device="" value="ADP2108AUJZ-3.3-R7"/>
 <part name="U5" library="flo-parts" deviceset="DCDC" device="" value="ADP2108AUJZ-1.8-R7"/>
-<part name="LED4" library="flo-led" deviceset="LED" device="KPT-2012" value="Green"/>
+<part name="LED4" library="flo-led" deviceset="LED" device="KPT-2012-E" value="Green"/>
 <part name="U$48" library="supply3" deviceset="+5V" device=""/>
 <part name="U$59" library="supply3" deviceset="VCCIO" device=""/>
 <part name="U$60" library="supply3" deviceset="GND" device=""/>
-<part name="LED3" library="flo-led" deviceset="LED" device="KPT-2012" value="Red"/>
+<part name="LED3" library="flo-led" deviceset="LED" device="KPT-2012-E" value="Red"/>
 <part name="U$61" library="supply3" deviceset="VCCIO" device=""/>
 <part name="JTX" library="flo-parts" deviceset="RESISTOR" device="CONNECT" value="0"/>
@@
 <part name="U$77" library="supply3" deviceset="GND" device=""/>
 <part name="U$19" library="flo-header" deviceset="CON2X2" device="PIN_L"/>
-<part name="U$21" library="flo-header" deviceset="CON1X1" device="PIN_XL"/>
-<part name="U$27" library="flo-header" deviceset="CON1X2" device="PIN_XL" value="CON1X2PIN_XL"/>
+<part name="S1" library="flo-header" deviceset="CON1X1" device="PIN_XL"/>
+<part name="S2" library="flo-header" deviceset="CON1X2" device="PIN_XL" value="CON1X2PIN_XL"/>
 <part name="U$46" library="supply3" deviceset="GND" device=""/>
-<part name="U$10" library="flo-header" deviceset="CON1X1" device="PIN_XL"/>
-<part name="U$11" library="flo-header" deviceset="CON1X1" device="PIN_XL"/>
+<part name="S4" library="flo-header" deviceset="CON1X1" device="PIN_XL"/>
+<part name="S3" library="flo-header" deviceset="CON1X1" device="PIN_XL"/>
 <part name="U$20" library="flo-parts" deviceset="TANTAL" device="1206"/>
 <part name="R7" library="flo-parts" deviceset="RESISTOR" device="WIDE" value="60"/>
@@
 <instance part="U$77" gate="G$1" x="213.36" y="58.42" rot="R180"/>
 <instance part="U$19" gate="G$1" x="195.58" y="22.86"/>
-<instance part="U$21" gate="G$1" x="-71.12" y="-50.8" rot="R180"/>
-<instance part="U$27" gate="G$1" x="-22.86" y="-33.02" rot="R270"/>
+<instance part="S1" gate="G$1" x="-71.12" y="-50.8" rot="R180"/>
+<instance part="S2" gate="G$1" x="-22.86" y="-33.02" rot="R270"/>
 <instance part="U$46" gate="G$1" x="170.18" y="60.96" rot="R180"/>
-<instance part="U$10" gate="G$1" x="43.18" y="-55.88" rot="R180"/>
-<instance part="U$11" gate="G$1" x="86.36" y="-55.88" rot="R180"/>
+<instance part="S4" gate="G$1" x="43.18" y="-55.88" rot="R180"/>
+<instance part="S3" gate="G$1" x="86.36" y="-55.88" rot="R180"/>
 <instance part="U$20" gate="G$1" x="-22.86" y="33.02" rot="R270"/>
 <instance part="R7" gate="R$1" x="195.58" y="-40.64"/>
@@
 <wire x1="-33.02" y1="-35.56" x2="-33.02" y2="-50.8" width="0.1524" layer="91"/>
 <label x="-33.02" y="-50.8" size="1.778" layer="95" rot="R90"/>
-<pinref part="U$27" gate="G$1" pin="P$2"/>
+<pinref part="S2" gate="G$1" pin="P$2"/>
 </segment>
 <segment>
@@
 <pinref part="U1" gate="NPN" pin="B"/>
 <wire x1="-66.04" y1="-50.8" x2="-73.66" y2="-50.8" width="0.1524" layer="91"/>
-<pinref part="U$21" gate="G$1" pin="P$1"/>
+<pinref part="S1" gate="G$1" pin="P$1"/>
 </segment>
 </net>
@@
 <wire x1="53.34" y1="-55.88" x2="40.64" y2="-55.88" width="0.1524" layer="91"/>
 <junction x="53.34" y="-55.88"/>
-<pinref part="U$10" gate="G$1" pin="P$1"/>
+<pinref part="S4" gate="G$1" pin="P$1"/>
 </segment>
 </net>
@@
 <wire x1="93.98" y1="-55.88" x2="83.82" y2="-55.88" width="0.1524" layer="91"/>
 <junction x="93.98" y="-55.88"/>
-<pinref part="U$11" gate="G$1" pin="P$1"/>
+<pinref part="S3" gate="G$1" pin="P$1"/>
 </segment>
 </net>
@@
 <pinref part="U1" gate="PNP" pin="B"/>
 <wire x1="-20.32" y1="-35.56" x2="-12.7" y2="-35.56" width="0.1524" layer="91"/>
-<pinref part="U$27" gate="G$1" pin="P$1"/>
-</segment>
-</net>
+<pinref part="S2" gate="G$1" pin="P$1"/>
+</segment>
+</net>
